File: colorsorter_schematic/colorsorter_schematic.kicad_sch (KiCad schematic)
At the start: 34 parts, among them J1 Conn_01x03_Pin, J2 Conn_01x03_Pin, J3 Conn_01x03_Pin, J4 Conn_01x05_Pin, J5 Conn_01x05_Pin, J6 Conn_01x03_Pin, J7 Conn_01x03_Pin, J8 Conn_01x02_Pin, SW1 SW_SPDT, U1 PIC24FJ64GA702-I/SO, U2 ESP8266-01_ESP-01, U3 LM1117DT-3.3/NOPB, Y1 830003156B

Commit message: J5 conn changed from 5 pin to 6 pin - updated pcb - saved changes
Parts:
- removed J5: Conn_01x05_Pin, Connector_PinHeader_2.54mm:PinHeader_1x05_P2.54mm_Vertical, symbol Connector:Conn_01x05_Pin
- added J5: Conn_01x06_Pin, Connector_PinHeader_2.54mm:PinHeader_1x06_P2.54mm_Vertical, symbol Connector:Conn_01x06_Pin
Connections:
- net GND: now also J5.6 (Pin_6)
- net SCL: now also J5.4 (Pin_4)
- net SDA: now also J5.3 (Pin_3)
- net at C1.2, C10.1, C11.2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: now also J5.5 (Pin_5)
- net at C2.1 (+), C7.2, J1.2 (Pin_2)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: now also J5.1 (Pin_1)
- net at U1.21 (PGD2/TDI/RP10/OCM1C/CTED11/RB10): now also J5.2 (Pin_2)
Changed lines of the file:
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@@
 	)
 	(junction
+		(at 198.12 20.32)
+		(diameter 0)
+		(color 0 0 0 0)
+	)
+	(junction
 		(at 31.75 91.44)
 		(diameter 0)
@@
 	(wire
 		(pts
+			(xy 265.43 68.58) (xy 265.43 20.32)
+		)
+		(stroke
+			(width 0)
+			(type default)
+		)
+	)
+	(wire
+		(pts
 			(xy 205.74 88.9) (xy 205.74 66.04)
 		)
@@
 	(wire
 		(pts
+			(xy 259.08 99.06) (xy 259.08 68.58)
+		)
+		(stroke
+			(width 0)
+			(type default)
+		)
+	)
+	(wire
+		(pts
 			(xy 97.79 128.27) (xy 224.79 128.27)
 		)
@@
 	(wire
 		(pts
+			(xy 265.43 20.32) (xy 198.12 20.32)
+		)
+		(stroke
+			(width 0)
+			(type default)
+		)
+	)
+	(wire
+		(pts
 			(xy 207.01 148.59) (xy 207.01 137.16)
 		)
@@
 	(wire
 		(pts
+			(xy 259.08 68.58) (xy 265.43 68.58)
+		)
+		(stroke
+			(width 0)
+			(type default)
+		)
+	)
+	(wire
+		(pts
 			(xy 39.37 88.9) (xy 39.37 86.36)
 		)
@@
 	)
 	(symbol
+		(lib_id "Connector:Conn_01x06_Pin")
+		(at 264.16 104.14 0)
+		(mirror y)
+		(unit 1)
+		(exclude_from_sim no)
+		(in_bom yes)
+		(on_board yes)
+		(dnp no)
+		(fields_autoplaced yes)
+		(property "Reference" "J5"
+			(at 265.43 104.1399 0)
+			(effects
+				(font
+					(size 1.27 1.27)
+				)
+				(justify right)
+			)
+		)
+		(property "Value" "Conn_01x06_Pin"
+			(at 265.43 106.6799 0)
+			(effects
+				(font
+					(size 1.27 1.27)
+				)
+				(justify right)
+			)
+		)
+		(property "Footprint" "Connector_PinHeader_2.54mm:PinHeader_1x06_P2.54mm_Vertical"
+			(at 264.16 104.14 0)
+			(effects
+				(font
+					(size 1.27 1.27)
+				)
+				(hide yes)
+			)
+		)
+		(property "Datasheet" "~"
+			(at 264.16 104.14 0)
+			(effects
+				(font
+					(size 1.27 1.27)
+				)
+				(hide yes)
+			)
+		)
+		(property "Description" "Generic connector, single row, 01x06, script generated"
+			(at 264.16 104.14 0)
+			(effects
+				(font
+					(size 1.27 1.27)
+				)
+				(hide yes)
+			)
+		)
+		(pin "4"
+		)
+		(pin "5"
+		)
+		(pin "1"
+		)
+		(pin "2"
+		)
+		(pin "6"
+		)
+		(pin "3"
+		)
+		(instances
+			(project ""
+				(path "/f85b107f-670e-4885-9436-e3b5bb042aa6"
+					(reference "J5")
+					(unit 1)
+				)
+			)
+		)
+	)
+	(symbol
 		(lib_id "power:GND")
 		(at 146.05 52.07 0)
@@
 					(unit 1)
 				)
-			)
-		)
-	)
-	(symbol
-		(lib_id "Connector:Conn_01x05_Pin")
-		(at 264.16 106.68 0)
-		(mirror y)
-		(unit 1)
-		(exclude_from_sim no)
-		(in_bom yes)
-		(on_board yes)
-		(dnp no)
-		(fields_autoplaced yes)
-		(property "Reference" "J5"
-			(at 265.43 105.4099 0)
-			(effects
-				(font
-					(size 1.27 1.27)
-				)
-				(justify right)
-			)
-		)
-		(property "Value" "Conn_01x05_Pin"
-			(at 265.43 107.9499 0)
-			(effects
-				(font
-					(size 1.27 1.27)
-				)
-				(justify right)
-				(hide yes)
-			)
-		)
-		(property "Footprint" "Connector_PinHeader_2.54mm:PinHeader_1x05_P2.54mm_Vertical"
-			(at 264.16 106.68 0)
-			(effects
-				(font
-					(size 1.27 1.27)
-				)
-				(hide yes)
-			)
-		)
-		(property "Datasheet" "~"
-			(at 264.16 106.68 0)
-			(effects
-				(font
-					(size 1.27 1.27)
-				)
-				(hide yes)
-			)
-		)
-		(property "Description" "Generic connector, single row, 01x05, script generated"
-			(at 264.16 106.68 0)
-			(effects
-				(font
-					(size 1.27 1.27)
-				)
-				(hide yes)
-			)
-		)
-		(pin "3"
-		)
-		(pin "2"
-		)
-		(pin "4"
-		)
-		(pin "1"
-		)
-		(pin "5"
-		)
-		(instances
-			(project ""
-				(path "/f85b107f-670e-4885-9436-e3b5bb042aa6"
-					(reference "J5")
-					(unit 1)
-				)

Commit message: Dodavanje izmjena na pcb projekta
Connections:
- net GND: now also J5.5 (Pin_5); no longer J5.6 (Pin_6)
- net SCL: now also J5.3 (Pin_3); no longer J5.4 (Pin_4)
- net at C1.2, C10.1, C11.2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: now also J5.4 (Pin_4); no longer J5.5 (Pin_5)
- net at C2.1 (+), C7.2, J1.2 (Pin_2)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: now also J5.6 (Pin_6); no longer J5.1 (Pin_1)
- net at U1.21 (PGD2/TDI/RP10/OCM1C/CTED11/RB10): now also J5.1 (Pin_1); no longer J5.2 (Pin_2)
- net SDA: no longer names the net of U1.18 (TDO/C1INC/C2INC/C3INC/TMPRN/RP9/SDA1/T1CK/CTED4/RB9)
- net SDA: now also J5.2 (Pin_2); no longer J5.3 (Pin_3)
Changed lines of the file:
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@@
+	(wire
+		(pts
+			(xy 259.08 101.6) (xy 252.73 101.6)
+		)
+		(stroke
+			(width 0)
+			(type default)
+		)
+	)
+	(wire
+		(pts
+			(xy 259.08 106.68) (xy 256.54 106.68)
+		)
+		(stroke
+			(width 0)
+			(type default)
+		)
+	)
 	(wire
 		(pts
@@
 	(wire
 		(pts
+			(xy 259.08 114.3) (xy 259.08 130.81)
+		)
+		(stroke
+			(width 0)
+			(type default)
+		)
+	)
+	(wire
+		(pts
 			(xy 99.06 22.86) (xy 99.06 25.4)
 		)
@@
 	(wire
 		(pts
+			(xy 255.27 104.14) (xy 255.27 106.68)
+		)
+		(stroke
+			(width 0)
+			(type default)
+		)
+	)
+	(wire
+		(pts
 			(xy 265.43 68.58) (xy 265.43 20.32)
 		)
@@
 	(wire
 		(pts
-			(xy 259.08 109.22) (xy 252.73 109.22)
+			(xy 259.08 95.25) (xy 259.08 68.58)
 		)
 		(stroke
@@
 	(wire
 		(pts
+			(xy 257.81 114.3) (xy 257.81 109.22)
+		)
+		(stroke
+			(width 0)
+			(type default)
+		)
+	)
+	(wire
+		(pts
 			(xy 142.24 134.62) (xy 142.24 137.16)
 		)
@@
 	(wire
 		(pts
+			(xy 256.54 109.22) (xy 252.73 109.22)
+		)
+		(stroke
+			(width 0)
+			(type default)
+		)
+	)
+	(wire
+		(pts
 			(xy 198.12 63.5) (xy 205.74 63.5)
 		)
@@
 	(wire
 		(pts
+			(xy 254 95.25) (xy 259.08 95.25)
+		)
+		(stroke
+			(width 0)
+			(type default)
+		)
+	)
+	(wire
+		(pts
 			(xy 167.64 34.29) (xy 179.07 34.29)
 		)
@@
 	(wire
 		(pts
+			(xy 257.81 109.22) (xy 259.08 109.22)
+		)
+		(stroke
+			(width 0)
+			(type default)
+		)
+	)
+	(wire
+		(pts
 			(xy 100.33 35.56) (xy 100.33 34.29)
 		)
@@
 	(wire
 		(pts
-			(xy 259.08 111.76) (xy 259.08 130.81)
-		)
-		(stroke
-			(width 0)
-			(type default)
-		)
-	)
-	(wire
-		(pts
 			(xy 209.55 71.12) (xy 209.55 72.39)
 		)
@@
 	(wire
 		(pts
+			(xy 251.46 99.06) (xy 251.46 101.6)
+		)
+		(stroke
+			(width 0)
+			(type default)
+		)
+	)
+	(wire
+		(pts
 			(xy 97.79 116.84) (xy 97.79 128.27)
 		)
@@
 	(wire
 		(pts
-			(xy 199.39 101.6) (xy 259.08 101.6)
+			(xy 199.39 101.6) (xy 251.46 101.6)
 		)
 		(stroke
@@
 	(wire
 		(pts
+			(xy 259.08 104.14) (xy 255.27 104.14)
+		)
+		(stroke
+			(width 0)
+			(type default)
+		)
+	)
+	(wire
+		(pts
 			(xy 209.55 86.36) (xy 215.9 86.36)
 		)
@@
 	(wire
 		(pts
+			(xy 259.08 99.06) (xy 251.46 99.06)
+		)
+		(stroke
+			(width 0)
+			(type default)
+		)
+	)
+	(wire
+		(pts
 			(xy 146.05 50.8) (xy 146.05 52.07)
 		)
@@
 	(wire
 		(pts
+			(xy 259.08 111.76) (xy 254 111.76)
+		)
+		(stroke
+			(width 0)
+			(type default)
+		)
+	)
+	(wire
+		(pts
 			(xy 198.12 20.32) (xy 198.12 52.07)
 		)
@@
 	(wire
 		(pts
+			(xy 256.54 106.68) (xy 256.54 109.22)
+		)
+		(stroke
+			(width 0)
+			(type default)
+		)
+	)
+	(wire
+		(pts
 			(xy 252.73 115.57) (xy 246.38 115.57)
 		)
@@
 	(wire
 		(pts
+			(xy 259.08 114.3) (xy 257.81 114.3)
+		)
+		(stroke
+			(width 0)
+			(type default)
+		)
+	)
+	(wire
+		(pts
 			(xy 86.36 99.06) (xy 86.36 40.64)
 		)
@@
 	(wire
 		(pts
-			(xy 232.41 106.68) (xy 259.08 106.68)
+			(xy 232.41 106.68) (xy 255.27 106.68)
 		)
 		(stroke
@@
 	(wire
 		(pts
-			(xy 259.08 99.06) (xy 259.08 68.58)
-		)
-		(stroke
-			(width 0)
-			(type default)
-		)
-	)
-	(wire
-		(pts
 			(xy 97.79 128.27) (xy 224.79 128.27)
 		)
@@
 	(wire
 		(pts
+			(xy 252.73 101.6) (xy 252.73 104.14)
+		)
+		(stroke
+			(width 0)
+			(type default)
+		)
+	)
+	(wire
+		(pts
 			(xy 246.38 115.57) (xy 246.38 116.84)
 		)
@@
 	(wire
 		(pts
-			(xy 228.6 104.14) (xy 259.08 104.14)
+			(xy 228.6 104.14) (xy 252.73 104.14)
 		)
 		(stroke
@@
 		)
 		(stroke
+			(width 0)
+			(type default)
+		)
+	)
+	(wire
+		(pts
+			(xy 254 111.76) (xy 254 95.25)
+		)
+		(stroke
