File: colorsorter_schematic/colorsorter_schematic.kicad_sch (KiCad schematic)
At the start: 34 parts, among them J1 Conn_01x03_Pin, J2 Conn_01x03_Pin, J3 Conn_01x03_Pin, J4 Conn_01x05_Pin, J5 Conn_01x06_Pin, J6 Conn_01x03_Pin, J7 Conn_01x03_Pin, J8 Conn_01x02_Pin, SW1 SW_SPDT, U1 PIC24FJ64GA702-I/SO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

Commit message: Final version PCB and manufacturing files
Parts:
- SW1: footprint twostateswitch:SLW12768644AD -> two_state_switch:SLW12768644AD
Changed lines of the file:
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@@
 			)
 		)
-		(property "Footprint" "twostateswitch:SLW12768644AD"
+		(property "Footprint" "two_state_switch:SLW12768644AD"
 			(at 48.26 83.82 0)
 			(effects
